File: Electronics/Boccia-controller/controller.sch (EAGLE design)
At the start: 24 parts

Commit message: Updated electronics schematics
Parts:
- removed POT_HEIGHT: (no value), rcl:R-TRIMM64X
- added F1, F2, F3, F4: FUSEBLANK_5X20MM, fuse:FUSEBLANK_5X20MM
- added POT_ELEVATION: (no value), rcl:R-TRIMM64X
Connections:
- removed net DIR_NEMA24: B1.51
- removed net N$27: B1.A2, POT_INCLINE.S
- removed net PUL_NEMA24: B1.50
- new net N$29: DRIVER_ROTATION.VCC, F4.2
- new net N$30: F3.2, REGULATOR_ELEVATION.VIN
- new net N$8: B1.A3, POT_ELEVATION.S
- new net N$9: B1.A4, POT_INCLINE.S
- net +24V: now also F1.1, F2.1, F3.1, F4.1; no longer REGULATOR_ELEVATION.VIN, REGULATOR_INCLINE.VIN, REGULATOR_RELEASE.VIN
- net N$28: now also F1.2, REGULATOR_RELEASE.VIN; no longer B1.A3, POT_HEIGHT.S
- net N$7: now also F2.2, REGULATOR_INCLINE.VIN; no longer DRIVER_ROTATION.VCC
- net PE: now also POT_ELEVATION.A; no longer POT_HEIGHT.A
- net V5_LOGIC: now also POT_ELEVATION.E; no longer POT_HEIGHT.E
Other:
- moved on the sheet: POT_INCLINE

Commit message: Updated new files with filters for optical sensors
Parts:
- added C4, C5, C6: 1nF, rcl:EL-BI35-12AXIAL
- added R3, R5, R6: 15k, rcl:R-US_R0805
Connections:
- new net N$27: OPTICAL_RELEASE.COL, R3.2
- new net N$31: OPTICAL_ROTATION_1.COL, R5.2
- new net N$32: OPTICAL_ROTATION_2.COL, R6.2
- net INTERRUPT_RELEASE: now also C4.1, R3.1; no longer OPTICAL_RELEASE.COL
- net INTERRUPT_ROTATION_1: now also C5.1, R5.1; no longer OPTICAL_ROTATION_1.COL
- net INTERRUPT_ROTATION_2: now also C6.1, R6.1; no longer OPTICAL_ROTATION_2.COL
- net PE: now also C4.2, C5.2, C6.2
Other:
- moved on the sheet: OPTICAL_ROTATION_2
